File: Hardware/Main Board - Single v20_v4.sch (EAGLE design)
At the start: 84 parts, among them J1 MICROMOD-2222-C, J10 MICRO-SD-PUSH-PUSH-EXT-PIN, J2 Vertical Qwiic Connector, J4 QWIIC_RIGHT_ANGLE, J5 CORTEX_JTAG_DEBUG_MINIMUM_PTH, J6 MICROMOD_FUNCTION_MAIN, Q1 3.1A/30V/105mΩ, Q2 20V/4.2A/52mΩ/1.4W, U1 STG3856QTR, U2 MCP73831, U3 ESD Diode, U4 AP7347DQ-33W5-7K-3.3V, U5 AP7361C-33

Commit message: Rolls version to v20
Other:
- note added: "v20"
- note removed: "v11"
Changed lines of the file:
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@@
 <text x="96.774" y="123.952" size="2.54" layer="94" font="vector" align="center">Function Board Connectors</text>
 <text x="95.25" y="271.526" size="2.54" layer="94" font="vector" align="center">Processor Board Connector</text>
-<text x="424.18" y="7.62" size="2.54" layer="94" font="vector" align="center">v11</text>
+<text x="424.18" y="7.62" size="2.54" layer="94" font="vector" align="center">v20</text>
 <wire x1="365.76" y1="132.08" x2="330.2" y2="132.08" width="0.2032" layer="97" style="longdash"/>
 <wire x1="330.2" y1="132.08" x2="284.48" y2="132.08" width="0.2032" layer="97" style="longdash"/>

Commit message: * Adds 4-pin header for other DFU lines
* Updates silk
* Uses VIN as power supply to battery charger
* Fixes PCH Mosfet
* Fixes polygons where applicable
* Adds SparkFun logo to topside.
Parts:
- removed R16: 2.2M, SparkFun-Resistors:2.2MOHMS-0603-1/10W-1%
- added J7: (no value), SparkFun-Connectors:CONN_041X04_NO_SILK
Connections:
- net I2C_SDA1-PROCESSOR/!SD_DISABLE! renamed I2C_SDA1-PROCESSOR/!SD_ENABLE!
- removed net !DFU-FC1!: R12.1, U1.2IN
- removed net N$1: 3V3_MEAS.1, C11.1, C9.1, R16.2, U5.OUT
- new net 1S2_MULTIPLEXER: J7.1, U1.1S2
- new net 2IN_MULTIPLEXER: J7.3, R12.1, U1.2IN
- new net 2S2_MULTIPLEXER: J7.2, U1.2S2
- new net 3V3_MEAS: 3V3_MEAS.1, C11.1, C9.1, U5.OUT
- net !BOOT!: now also J6.DFU_!BOOT!; no longer J6.MCU_!BOOT!
- net !DFU-FC0!: now also J6.DFU_!ACTIVE!; no longer J6.MCU_!DFU_STAT!
- net !RESET!: now also J6.DFU_!RST!; no longer J6.MCU_!RST!
- net 3.3V: no longer R19.2
- net GND: now also J7.4, R19.2; no longer R16.1
- net RX1-DFU_TX-FC0-PLEX: now also J6.DFU_FC_TX; no longer J6.MCU_DFU_TX
- net TX1-DFU_RX-FC0-PLEX: now also J6.DFU_FC_RX; no longer J6.MCU_DFU_RX
- net VCC: no longer C3.1, R5.1, U2.VIN
- net VIN: now also C3.1, R5.1, U2.VIN
Other:
- note added: "Cut trace to remove resistor divider. Good for deep sleep power considerations."
- moved on the sheet: 3V3_MEAS, DIVIDER, J1, R10, R7
